Commit message: URDF loader
Attempted to write custom URDF loader using tinyxml2.
Was able to extract URDF loading code from Bullet examples.

File: data/cyton_gamma_1500/cyton_gamma_1500.urdf (robot description, URDF)
Before this commit: robot cyton_gamma_1500, 12 links, 11 joints
Links:
- link base_link: geometry collision box size=0.154 0.177 0.094; visual mesh filename=meshes/base.dae
- link elbow_pitch: geometry collision box size=0.0549 0.1557 0.076; visual mesh filename=meshes/elbow_pitch.dae
- link elbow_yaw: geometry collision box size=0.0535 0.1160 0.0402; visual mesh filename=meshes/elbow_yaw.dae
- link gripper_finger1: geometry collision box size=0.015 0.0229 0.0475; visual mesh filename=meshes/gripper_finger1.dae
- link gripper_finger2: geometry collision box size=0.015 0.0229 0.0475; visual mesh filename=meshes/gripper_finger2.dae
- link shoulder_pitch: geometry collision box size=0.0709 0.19363 0.083; visual mesh filename=meshes/shoulder_pitch.dae
- link shoulder_roll: geometry collision box size=0.09829 0.18143 0.08392; visual mesh filename=meshes/shoulder_roll.dae
- link shoulder_yaw: geometry collision box size=0.0717 0.1846 0.0756; visual mesh filename=meshes/shoulder_yaw.dae
- link wrist_pitch: geometry collision box size=0.026 0.0435 0.05185; visual mesh filename=meshes/wrist_pitch.dae
- link wrist_roll: geometry collision box size=0.0518 0.0723 0.1004; visual mesh filename=meshes/wrist_roll.dae
